Commit message: feat(sim): improve MuJoCo physics & collision
- Physics: add timestep=0.001, noslip_iterations=5, elliptic friction cone
  for stable contact-rich grasping
- Gripper collision: add fixed jaw finger, palm back-plate, moving jaw
  full-coverage proxies with high-friction contact parameters
- Banana: replace box with capsule collision proxy matching real cross-section;
  add free-joint damping=5.0 to damp contact oscillations
- Scene layout: reposition robot base, table, curtain, banana for better
  pick-and-place workspace; stiffen table contact (solref=0.003)
- Camera: reposition wrist camera to palm back-plate center aimed at jaw
  closing center

File: src/robot_description/urdf/lerobot/so101/so101_cameras.xacro (robot description, xacro)
@@ -2,5 +2,5 @@
 <robot xmlns:xacro="http://www.ros.org/wiki/xacro">
     <!-- ============================================= -->
-    <!-- Wrist Camera (mounted on gripper/wrist link) -->
+    <!-- Wrist Camera (mounted on gripper body)      -->
     <!-- ============================================= -->
     <link name="wrist_camera_link">
@@ -14,6 +14,6 @@
         <parent link="gripper"/>
         <child link="wrist_camera_link"/>
-        <!-- Position camera in front of gripper, pointing downward -->
-        <origin xyz="0.05 0.0 0.0" rpy="0 0.5 0"/>
+        <!-- Camera at center of palm back-plate, aimed at jaw closing center -->
+        <origin xyz="0.002 0.061 -0.025" rpy="-3.14159 -0.4 -1.5708"/>
     </joint>
     <!-- Wrist Camera Sensor for Gazebo -->
@@ -22,5 +22,5 @@
             <update_rate>30</update_rate>
             <camera>
-                <horizontal_fov>1.047</horizontal_fov>  <!-- 60 degrees -->
+                <horizontal_fov>1.5708</horizontal_fov>  <!-- 90 degrees -->
                 <image>
                     <width>640</width>
@@ -29,5 +29,5 @@
                 </image>
                 <clip>
-                    <near>0.1</near>
+                    <near>0.01</near>
                     <far>100</far>
                 </clip>
