Commit message: feat(sim): align Gazebo/MuJoCo cameras, assets and lighting
Add camera_presets.py with platform-specific default camera poses so
that a single YAML config (use_default_transform: true) works for both
Gazebo and MuJoCo without manual coordinate conversion.

Update pick_banana Gazebo world template to match layout.yaml canonical
values (table scale 0.156, banana x=0, curtain yaw flip, ground z).

Tune MuJoCo lighting: reduce headlight diffuse, use single shadow-
casting directional light, add low-specular materials for table and
robot to eliminate top-camera overexposure.

Add Gazebo material overrides in so101_gazebo.xacro so the robot arm
renders with correct colors instead of default grey.

Signed-off-by: $(git config user.name) <$(git config user.email)>
Signed-off-by: grangerxsp <xingshiping@huawei.com>

File: src/robot_description/urdf/lerobot/so101/so101_gazebo.xacro (robot description, xacro)
@@ -9,3 +9,24 @@
         </plugin>
     </gazebo>
+    <!-- ============================================= -->
+    <!-- Gazebo material: uniform dark (sts3215 black) -->
+    <!-- ============================================= -->
+    <!-- Gazebo cannot color individual visuals within a link separately.
+         Uniform black matches the real robot's dominant visual appearance. -->
+    <xacro:macro name="gz_black" params="link_name">
+        <gazebo reference="${link_name}">
+            <visual><material>
+                <ambient>0.12 0.12 0.12 1</ambient>
+                <diffuse>0.12 0.12 0.12 1</diffuse>
+                <specular>0.15 0.15 0.15 1</specular>
+            </material></visual>
+        </gazebo>
+    </xacro:macro>
+    <xacro:gz_black link_name="base"/>
+    <xacro:gz_black link_name="shoulder"/>
+    <xacro:gz_black link_name="upper_arm"/>
+    <xacro:gz_black link_name="lower_arm"/>
+    <xacro:gz_black link_name="wrist"/>
+    <xacro:gz_black link_name="gripper"/>
+    <xacro:gz_black link_name="jaw"/>
 </robot>
